File: KiCad/Proyecto_Final/Frontend.sch (KiCad schematic (older format))
At the start: 33 parts

Commit message: Avances de esquematico frontend
Other:
- note added: "50 Ohms"
Changed lines of the file:
@@
 Text Label 5900 5500 2    50   ~ 0
 REF_IN
+Text Notes 7100 2350 0    50   ~ 10
+50 Ohms
+Text Notes 8200 3500 0    50   ~ 10
+50 Ohms
 $EndSCHEMATC

Commit message: Agregadas librerias al repo para mejor portabilidad
Parts:
- T? (x2): symbol hackrf:BALUN_1-1 -> Frontend-rescue:BALUN_1-1-hackrf
- U?: footprint (none) -> Package_DFN_QFN:QFN-32-1EP_5x5mm_P0.5mm_EP3.7x3.7mm; symbol hackrf:RFFC5072 -> hackrf:hackrf_RFFC5072
Changed lines of the file:
@@
 $EndDescr
 $Comp
-L hackrf:RFFC5072 U?
+L hackrf:hackrf_RFFC5072 U?
 U 1 1 5FF11A11
 P 5700 3950
 F 0 "U?" H 5650 4050 60  0000 L CNN
 F 1 "RFFC5072" H 5500 3950 60  0000 L CNN
-F 2 "" H 5700 3950 60  0000 C CNN
-F 3 "" H 5700 3950 60  0000 C CNN
+F 2 "Package_DFN_QFN:QFN-32-1EP_5x5mm_P0.5mm_EP3.7x3.7mm" H 5700 3950 60  0001 C CNN
+F 3 "" H 5700 3950 60  0001 C CNN
 	1    5700 3950
 	1    0    0    -1
@@
 	5850 2800 5850 2550
 $Comp
-L hackrf:BALUN_1-1 T?
+L Frontend-rescue:BALUN_1-1-hackrf T?
 U 1 1 5FEE321F
 P 6300 2500
@@
 NoConn ~ 4550 3800
 $Comp
-L hackrf:BALUN_1-1 T?
+L Frontend-rescue:BALUN_1-1-hackrf T?
 U 1 1 5FEE1677
 P 7450 3650

Commit message: Agregadas y actualizadas librerias y esquematico frontend.
Parts:
- added C? (x3): 100pF, symbol Device:C
- added C? (x2): 33pF, symbol Device:C
- added FL?: DEA162690LT-5064A1, SamacSys_Parts:DEA162690LT5051B1, symbol SamacSys_Parts:DEA162690LT-5064A1
- added J?: Conn_Coaxial, Connector_Coaxial:SMA_Molex_73251-2120_EdgeMount_Horizontal, symbol Connector:Conn_Coaxial
- added U?: SKY13351, symbol gsg-symbols:SKY13351
- added U?: MAAL-010200, Package_TO_SOT_SMD:SOT-89-3, symbol Tesis2020-21:MAAL-010200
- T? (x2): symbol Frontend-rescue:BALUN_1-1-hackrf -> Frontend-rescue:BALUN_1-1-hackrf-Frontend-rescue
Connections:
- net labels added: Rx_Amp, Rx_Amp_Bypass
- wire segments 87 -> 107
Changed lines of the file:
@@
 	5850 2800 5850 2550
 $Comp
-L Frontend-rescue:BALUN_1-1-hackrf T?
+L Frontend-rescue:BALUN_1-1-hackrf-Frontend-rescue T?
 U 1 1 5FEE321F
 P 6300 2500
@@
 NoConn ~ 4550 3800
 $Comp
-L Frontend-rescue:BALUN_1-1-hackrf T?
+L Frontend-rescue:BALUN_1-1-hackrf-Frontend-rescue T?
 U 1 1 5FEE1677
 P 7450 3650
@@
 Text Notes 8200 3500 0    50   ~ 10
 50 Ohms
+$Comp
+L SamacSys_Parts:DEA162690LT-5064A1 FL?
+U 1 1 601D3384
+P 1750 8650
+F 0 "FL?" H 2350 9415 50  0000 C CNN
+F 1 "DEA162690LT-5064A1" H 2350 9324 50  0000 C CNN
+F 2 "SamacSys_Parts:DEA162690LT5051B1" H 1750 9800 50  0001 L CNN
+F 3 "https://product.tdk.com/info/en/documents/data_sheet/rf_lpf_dea162690lt-5064a1_en.pdf" H 1750 9700 50  0001 L CNN
+F 4 "Signal Conditioning Low Pass Filter for LTE" H 1750 9600 50  0001 L CNN "Description"
+F 5 "TDK" H 1750 9400 50  0001 L CNN "Manufacturer_Name"
+F 6 "DEA162690LT-5064A1" H 1750 9300 50  0001 L CNN "Manufacturer_Part_Number"
+	1    1750 8650
+	1    0    0    -1
+$EndComp
+$Comp
+L Connector:Conn_Coaxial J?
+U 1 1 601DB430
+P 950 8350
+F 0 "J?" H 878 8588 50  0000 C CNN
+F 1 "Conn_Coaxial" H 878 8497 50  0000 C CNN
+F 2 "Connector_Coaxial:SMA_Molex_73251-2120_EdgeMount_Horizontal" H 950 8350 50  0001 C CNN
+F 3 " ~" H 950 8350 50  0001 C CNN
+	1    950  8350
+	-1   0    0    -1
+$EndComp
+$Comp
+L power:GND #PWR?
+U 1 1 601E095C
+P 950 8550
+F 0 "#PWR?" H 950 8300 50  0001 C CNN
+F 1 "GND" H 955 8377 50  0000 C CNN
+F 2 "" H 950 8550 50  0001 C CNN
+F 3 "" H 950 8550 50  0001 C CNN
+	1    950  8550
+	1    0    0    -1
+$EndComp
+$Comp
+L power:GND #PWR?
+U 1 1 601E0CAC
+P 2250 8950
+F 0 "#PWR?" H 2250 8700 50  0001 C CNN
+F 1 "GND" H 2255 8777 50  0000 C CNN
+F 2 "" H 2250 8950 50  0001 C CNN
+F 3 "" H 2250 8950 50  0001 C CNN
+	1    2250 8950
+	1    0    0    -1
+$EndComp
+Wire Wire Line
+	2250 8950 2250 8850
+Wire Wire Line
+	2450 8850 2250 8850
+Connection ~ 2250 8850
+Wire Wire Line
+	1150 8350 1550 8350
+$Comp
+L gsg-symbols:SKY13351 U?
+U 1 1 601DE6A1
+P 4450 8350
+F 0 "U?" H 4450 8787 60  0000 C CNN
+F 1 "SKY13351" H 4450 8681 60  0000 C CNN
+F 2 "" H 4450 8350 60  0000 C CNN
+F 3 "" H 4450 8350 60  0000 C CNN
+	1    4450 8350
+	-1   0    0    -1
+$EndComp
+$Comp
+L Device:C C?
+U 1 1 601E89A6
+P 3600 8350
+F 0 "C?" V 3348 8350 50  0000 C CNN
+F 1 "100pF" V 3439 8350 50  0000 C CNN
+F 2 "" H 3638 8200 50  0001 C CNN
+F 3 "~" H 3600 8350 50  0001 C CNN
+	1    3600 8350
+	0    1    1    0
+$EndComp
+Wire Wire Line
+	3450 8350 3150 8350
+Wire Wire Line
+	3750 8350 4000 8350
+Wire Wire Line
+	4000 8250 3850 8250
+Wire Wire Line
+	4000 8450 3850 8450
+Text GLabel 3400 7450 0    50   Input ~ 0
+Rx_Amp
+Text GLabel 3650 8800 0    50   Input ~ 0
+Rx_Amp_Bypass
+$Comp
+L Device:C C?
+U 1 1 601F446A
+P 5250 8150
+F 0 "C?" V 4998 8150 50  0000 C CNN
+F 1 "100pF" V 5089 8150 50  0000 C CNN
+F 2 "" H 5288 8000 50  0001 C CNN
+F 3 "~" H 5250 8150 50  0001 C CNN
+	1    5250 8150
+	0    1    1    0
+$EndComp
+$Comp
+L Device:C C?
+U 1 1 601F4A10
+P 5250 8550
+F 0 "C?" V 4998 8550 50  0000 C CNN
+F 1 "100pF" V 5089 8550 50  0000 C CNN
+F 2 "" H 5288 8400 50  0001 C CNN
+F 3 "~" H 5250 8550 50  0001 C CNN
+	1    5250 8550
+	0    1    1    0
+$EndComp
+Wire Wire Line
+	4900 8250 4900 8150
+Wire Wire Line
+	4900 8150 5100 8150
+Wire Wire Line
+	4900 8450 4900 8550
+Wire Wire Line
+	4900 8550 5100 8550
+$Comp
+L power:GND #PWR?
+U 1 1 601FAAAB
+P 5000 8750
+F 0 "#PWR?" H 5000 8500 50  0001 C CNN
+F 1 "GND" H 5005 8577 50  0000 C CNN
+F 2 "" H 5000 8750 50  0001 C CNN
+F 3 "" H 5000 8750 50  0001 C CNN
+	1    5000 8750
+	1    0    0    -1
+$EndComp
+Wire Wire Line
+	5000 8750 5000 8350
+Wire Wire Line
+	5000 8350 4900 8350
+Wire Wire Line
+	3850 7450 3850 8250
+Wire Wire Line
+	3850 8800 3750 8800
+Wire Wire Line
+	3850 8450 3850 8800
+Wire Wire Line
+	3850 7450 3500 7450
+$Comp
+L Device:C C?
+U 1 1 602079FB
+P 3500 7600
+F 0 "C?" H 3615 7646 50  0000 L CNN
+F 1 "33pF" H 3615 7555 50  0000 L CNN
+F 2 "" H 3538 7450 50  0001 C CNN
+F 3 "~" H 3500 7600 50  0001 C CNN
+	1    3500 7600
+	1    0    0    -1
+$EndComp
+Connection ~ 3500 7450
+Wire Wire Line
+	3500 7450 3400 7450
+$Comp
+L Device:C C?
+U 1 1 602084F0
+P 3750 8950
+F 0 "C?" H 3865 8996 50  0000 L CNN
+F 1 "33pF" H 3865 8905 50  0000 L CNN
+F 2 "" H 3788 8800 50  0001 C CNN
+F 3 "~" H 3750 8950 50  0001 C CNN
+	1    3750 8950
+	1    0    0    -1
+$EndComp
+Connection ~ 3750 8800
+Wire Wire Line
+	3750 8800 3650 8800
+$Comp
+L power:GND #PWR?
+U 1 1 60208E42
+P 3750 9100
+F 0 "#PWR?" H 3750 8850 50  0001 C CNN
+F 1 "GND" H 3755 8927 50  0000 C CNN
+F 2 "" H 3750 9100 50  0001 C CNN
+F 3 "" H 3750 9100 50  0001 C CNN
+	1    3750 9100
+	1    0    0    -1
+$EndComp
+$Comp
+L power:GND #PWR?
+U 1 1 602090A0
+P 3500 7750
+F 0 "#PWR?" H 3500 7500 50  0001 C CNN
+F 1 "GND" H 3505 7577 50  0000 C CNN
+F 2 "" H 3500 7750 50  0001 C CNN
+F 3 "" H 3500 7750 50  0001 C CNN
+	1    3500 7750
+	1    0    0    -1
+$EndComp
+$Comp
+L Tesis2020-21:MAAL-010200 U?
+U 1 1 6020E695
+P 6100 8450
+F 0 "U?" H 6550 8999 50  0000 C CNN
+F 1 "MAAL-010200" H 6550 8916 39  0000 C CNN
+F 2 "Package_TO_SOT_SMD:SOT-89-3" H 6725 9000 50  0001 C CNN
+F 3 "" H 6200 8900 50  0001 C CNN
+	1    6100 8450
+	1    0    0    -1
+$EndComp
+Wire Wire Line
+	5400 8150 6000 8150
+$Comp
+L power:GND #PWR?
+U 1 1 60212C8F
+P 6550 8550
+F 0 "#PWR?" H 6550 8300 50  0001 C CNN
+F 1 "GND" H 6555 8377 50  0000 C CNN
+F 2 "" H 6550 8550 50  0001 C CNN
+F 3 "" H 6550 8550 50  0001 C CNN
+	1    6550 8550
+	1    0    0    -1
+$EndComp
 $EndSCHEMATC

Commit message: Actualizacion esquematico y carga de datasheets.
Parts:
- removed C? (x4): 100pF, symbol Device:C
- removed FL?: DEA162690LT-5064A1, SamacSys_Parts:DEA162690LT5051B1, symbol SamacSys_Parts:DEA162690LT-5064A1
- removed T? (x2): BALUN_1-1, symbol Frontend-rescue:BALUN_1-1-hackrf-Frontend-rescue
- added C? (x7): 100pF, symbol Device:C
- added C? (x6): 33pF, symbol Device:C
- added C?: 0.1uF, symbol Device:C
- added FL?: DEA162690LT-5064A1, SamacSys_Parts:DEA162690LT5051B1, symbol SamacSys_Parts:DEA162690LT-5064A1
- added L?: 12nH, symbol Device:L
- added Q?: IRLML0040TRPBF, SOT95P237X112-3N, symbol Tesis2020-21:IRLML0040TRPBF
- added R?: 10k, symbol Device:R
- added T? (x2): B0310J50100AHF, B0310J50100AHF, symbol Tesis2020-21:B0310J50100AHF
- added U? (x3): SKY13351, symbol gsg-symbols:SKY13351
Connections:
- net GND: now also C?.2, C?.2, C?.2, C?.2, C?.2, C?.2, C?.2, FL?.2 (GND_1), FL?.4 (GND_2), Q?.2 (S), R?.2, T?.2 (GND), T?.2 (GND), U?.2 (GND), U?.2 (GND), U?.2 (GND)
- net Rx_Amp: now also C?.1, U?.6 (VCTL1)
- net Rx_Amp_Bypass: now also C?.1, U?.4 (VCTL2)
- net VDD: now also C?.1, L?.1
- net at L?.2, U?.27 (MIX_OPN): now also T?.4 (BP2)
- net at U?.24 (MIX_IPN): now also T?.4 (BP2)
- net at U?.23 (MIX_IPP): now also T?.3 (BP1)
- net at L?.2, U?.28 (MIX_OPP): now also T?.3 (BP1)
- net at J?.1 (In): now also FL?.1 (IN/OUT_PORT)
- net at C?.2: now also FL?.3 (OUT/IN_PORT)
- net at C?.1: now also C?.2
- net at U?.3 (RF_OUT/VDD): now also C?.2
- new net: C?.1, U?.1 (OUT1) (x2)
- new net: C?.1, U?.3 (OUT2) (x2)
- new net: C?.2, U?.5 (INPUT) (x2)
- new net: C?.1, U?.5 (INPUT)
- new net: C?.2, U?.1 (OUT1)
- new net: C?.2, U?.3 (OUT2)
- new net: C?.1, T?.1 (UP)
- new net: C?.2, T?.1 (UP)
- new net !Rx_Amp: Q?.1 (G), R?.1
- new net !Rx_Mix: C?.1, C?.1, C?.1, U?.4 (VCTL2), U?.6 (VCTL1), U?.6 (VCTL1)
- new net RF_IN: C?.1
- new net Rx_Mix: C?.1, U?.4 (VCTL2)
Other:
- note added: "100 Ohms\nDiferencial"
- note added: "Al MAX2837"
- note added: "Al RFFC5072"
- note added: "SOLO RX"

Commit message: Añadidos datasheets y terminado esquematico frontend.
Parts:
- removed FL?: DEA162690LT-5064A1, SamacSys_Parts:DEA162690LT5051B1, symbol SamacSys_Parts:DEA162690LT-5064A1
- removed Q?: IRLML0040TRPBF, SOT95P237X112-3N, symbol Tesis2020-21:IRLML0040TRPBF
- added C?: 0.1uF, symbol Device:C
- added C?: 10nF, symbol Device:C
- added FL?: DEA162690LT-5064A1, SamacSys_Parts:DEA162690LT5051B1, symbol SamacSys_Parts:DEA162690LT-5064A1
- added Q?: BSS315P, SOT95P237X112-3N, symbol SamacSys_Parts:BSS315PH6327XTSA1
- C?: footprint (none) -> Capacitor_SMD:C_0402_1005Metric
- L?: footprint (none) -> Inductor_SMD:L_0402_1005Metric
Connections:
- net !Rx_Amp: now also R?.2, Q?.1; no longer R?.1
- net GND: now also C?.2, C?.2, FL?.2 (GND_1), FL?.4 (GND_2); no longer R?.2
- net VDD: now also R?.1, C?.1, Q?.2; no longer C?.1, L?.1
- net at J?.1 (In): now also FL?.1 (IN/OUT_PORT)
- net at C?.2: now also FL?.3 (OUT/IN_PORT)
- net at C?.2, U?.3 (RF_OUT/VDD): now also L?.2
- new net: C?.1, C?.1, L?.1, Q?.3
Other:
- moved on the sheet: C?, L?, R?

Commit message: Enumeración de componentes, asignación de footprints y netlist generada para frontend.
Parts:
- C1, C10, C11, C12, C13, C14, C15, C16, C17, C18, C19, C2, C20, C21, C22, C23, C24, C25, C26, C27, C28, C29, C3, C31, C32, C33, C34, C35, C36, C37, C38, C39, C4, C5, C6, C7, C8, C9: renamed from C?; footprint (none) -> Capacitor_SMD:C_0402_1005Metric
- D1: renamed from D?; footprint (none) -> LED_SMD:LED_0805_2012Metric
- L1, L2: renamed from L?; footprint (none) -> Inductor_SMD:L_0402_1005Metric
- Q1: renamed from Q?; footprint SOT95P237X112-3N -> SamacSys_Parts:SOT95P237X112-3N
- R1, R2, R3, R4, R5, R6: renamed from R?; footprint (none) -> Resistor_SMD:R_0805_2012Metric
- T1, T2: renamed from T?; footprint B0310J50100AHF -> SamacSys_Parts:B0310J50100AHF
- U1, U3, U4, U5: renamed from U?; footprint (none) -> gsg-modules:SKY13351-378LF
- gave numbers to parts that had none: 6
