File: KiCad/Proyecto_Final/Frontend.sch (KiCad schematic (older format))
At the start: 69 parts, among them J1 RF_IN, Q1 Si2301CDS, T1 B0310J50100AHF, T2 B0310J50100AHF, U1 SKY13351, U2 RFFC5072, U3 SKY13351, U4 SKY13351, U5 SKY13351, U6 SKY13351, U7 SKY13351, U8 MAAL-010200

Commit message: Avances PCB.
Parts:
- renumbered C37 to C100, C38 to C101, C39 to C102, C40 to C103, C41 to C104, C42 to C105, C43 to C106, C44 to C107, C45 to C108, C46 to C109, C47 to C110, C1 to C64, C2 to C65, C3 to C66, C4 to C67, C5 to C68, C6 to C69, C7 to C70, C8 to C71, C9 to C72, C10 to C73, C11 to C74, C12 to C75, C13 to C76, C14 to C77, C15 to C78, C16 to C79, C17 to C80, C18 to C81, C19 to C82, C20 to C83, C21 to C84, C22 to C85, C23 to C86, C24 to C87, C25 to C88, C26 to C89, C27 to C90, C28 to C91, C29 to C92, C30 to C93, C31 to C94, C32 to C95, C33 to C96, C34 to C97, C35 to C98, C36 to C99, J1 to J15, L1 to L2, L2 to L3, L3 to L4, R1 to R21, R2 to R22, R3 to R23, R4 to R24, R5 to R25, R6 to R26, T1 to T2, T2 to T3, U4 to U10, U5 to U11, U6 to U12, U7 to U13, U8 to U14, U1 to U7, U2 to U8, U3 to U9

Commit message: Avances librería mezclador.
Parts:
- removed C80: 33pF, Capacitor_SMD:C_0402_1005Metric, symbol Device:C
- removed R21: 10k, Resistor_SMD:R_0402_1005Metric, symbol Device:R
Connections:
- net RESETX: no longer names the net of U8.29 (RESETX)
- no-connect marks 7 -> 8
Changed lines of the file:
@@
-$EndComp
-$Comp
-L Device:C C80
-U 1 1 5FF2D567
-P 1150 3250
-F 0 "C80" H 1265 3296 50  0000 L CNN
-F 1 "33pF" H 1265 3205 50  0000 L CNN
-F 2 "Capacitor_SMD:C_0402_1005Metric" H 1188 3100 50  0001 C CNN
-F 3 "~" H 1150 3250 50  0001 C CNN
-	1    1150 3250
-	1    0    0    -1
-$EndComp
-$Comp
-L power:GND #PWR0100
-U 1 1 5FF2EC52
-P 1150 3400
-F 0 "#PWR0100" H 1150 3150 50  0001 C CNN
-F 1 "GND" H 1155 3227 50  0000 C CNN
-F 2 "" H 1150 3400 50  0001 C CNN
-F 3 "" H 1150 3400 50  0001 C CNN
-	1    1150 3400
-	1    0    0    -1
 $EndComp
 $Comp
@@
 	0    1    1    0
 $EndComp
-Text GLabel 6550 2300 0    50   Input ~ 0
-RESETX
 Text GLabel 6550 2450 0    50   Input ~ 0
 SPI1_CS0
@@
 Text GLabel 6550 2750 0    50   Input ~ 0
 SPI1_MOSI
-Text GLabel 1050 3050 0    50   Input ~ 0
-RESETX
 $Comp
 L Device:C C78
@@
 	6800 2450 6800 2800
 Wire Wire Line
-	6900 2800 6900 2300
-Wire Wire Line
-	6900 2300 6550 2300
-Wire Wire Line
 	7250 2650 7200 2650
 Wire Wire Line
@@
 Text GLabel 6700 5100 3    50   Input ~ 0
 REF_IN
-$Comp
-L Device:R R21
-U 1 1 60A036F9
-P 1150 2850
-F 0 "R21" H 1220 2896 50  0000 L CNN
-F 1 "10k" H 1220 2805 50  0000 L CNN
-F 2 "Resistor_SMD:R_0402_1005Metric" V 1080 2850 50  0001 C CNN
-F 3 "~" H 1150 2850 50  0001 C CNN
-	1    1150 2850
-	1    0    0    -1
-$EndComp
-$Comp
-L power:+3.3V #PWR093
-U 1 1 60A18487
-P 1150 2700
-F 0 "#PWR093" H 1150 2550 50  0001 C CNN
-F 1 "+3.3V" H 1165 2873 50  0000 C CNN
-F 2 "" H 1150 2700 50  0001 C CNN
-F 3 "" H 1150 2700 50  0001 C CNN
-	1    1150 2700
-	1    0    0    -1
-$EndComp
-Wire Wire Line
-	1150 3000 1150 3050
-Wire Wire Line
-	1050 3050 1150 3050
-Connection ~ 1150 3050
-Wire Wire Line
-	1150 3050 1150 3100
 Wire Wire Line
 	10650 7450 10550 7450
@@
 Wire Wire Line
 	7900 7050 7900 7400
+NoConn ~ 6900 2800
 $EndSCHEMATC

Commit message: comito
Parts:
- added C80: 33pF, Capacitor_SMD:C_0402_1005Metric, symbol Device:C
- added R23: 10k, Resistor_SMD:R_0402_1005Metric, symbol Device:R
- renumbered C71 to C68, C72 to C69, C68 to C70, C69 to C71, C70 to C72, J15 to J16, R22 to R24, R23 to R25, R24 to R26, R25 to R27, R26 to R28
Connections:
- net +3.3VA: now also C68.1, C69.1, C87.1, Q1.2 (S), R28.1, U8.19 (DIG_VDD)
- net +3V3: now also R23.1; no longer C68.1, C69.1, C87.1, Q1.2 (S), R28.1, U8.19 (DIG_VDD)
- net GND: now also C80.2
- net RESETX: now reaches U8.29 (RESETX)
- net RESETX: now also C80.1, R23.2
- no-connect marks 8 -> 7
Other:
- moved on the sheet: C68, C69

Commit message: Se cambiaron los switches de RF y se ajustó el PCB.
Parts:
- removed U10, U11, U12, U13, U7, U9: SKY13351, gsg-modules:SKY13351-378LF, symbol gsg-symbols:SKY13351
- added IC1, IC2, IC3, IC4, IC5, IC6: SKY13335-381LF, SamacSys_Parts:SON50P200X150X50-7N, symbol SamacSys_Parts:SKY13335-381LF
- renumbered C106 to C105, C105 to C106, J16 to J18, U8 to U7, U14 to U8
Connections:
- net Filt_Bypass: now also IC2.4 (VCTL2), IC3.6 (VCTL1)
- net Filtro: now also IC2.6 (VCTL1), IC3.4 (VCTL2)
- net GND: now also IC1.2 (GND), IC1.7 (EP), IC2.2 (GND), IC2.7 (EP), IC3.2 (GND), IC3.7 (EP), IC4.2 (GND), IC4.7 (EP), IC5.2 (GND), IC5.7 (EP), IC6.2 (GND), IC6.7 (EP)
- net Rx_Amp: now also IC4.4 (VCTL2), IC5.6 (VCTL1)
- net Rx_Amp_Bypass: now also IC4.6 (VCTL1), IC5.4 (VCTL2)
- net Rx_Mix: now also IC1.4 (VCTL2), IC6.4 (VCTL2)
- net Rx_Mix_Bypass: now also IC1.6 (VCTL1), IC6.6 (VCTL1)
- net SWITCH: now also IC1.1 (OUT1)
- net at C102.2: now also IC4.1 (OUT1)
- net at C96.2: now also IC4.3 (OUT2)
- net at C100.1: now also IC4.5 (RFC)
- net at C100.2: now also IC3.5 (RFC)
- net at C97.1: now also IC5.1 (OUT1)
- net at C102.1: now also IC5.3 (OUT2)
- net at C101.2: now also IC5.5 (RFC)
- net at C101.1: now also IC6.5 (RFC)
- net at C98.2: now also IC6.1 (OUT1)
- net at C103.2: now also IC6.3 (OUT2)
- net at C74.1: now also IC1.3 (OUT2)
- net at C73.2: now also IC1.5 (RFC)
- net at C109.2: now also IC2.1 (OUT1)
- net at C99.2: now also IC2.3 (OUT2)
- net at C88.1: now also IC2.5 (RFC)
- net at C99.1: now also IC3.1 (OUT1)
- net at C110.1: now also IC3.3 (OUT2)
Other:
- moved on the sheet: C100, C101, C103, C104, C105, C106, C107, C70, C73, C75, C88, C96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

Commit message: Agregados capacitores de balunes faltantes
Parts:
- added C111, C112: 100nF, Capacitor_SMD:C_0402_1005Metric, symbol Device:C
Connections:
- net GND: now also C111.2, C112.2; no longer T2.2 (GND), T3.2 (GND)
- new net: C112.1, T3.2 (GND)
- new net: C111.1, T2.2 (GND)
Changed lines of the file:
@@
 L power:GND #PWR0144
 U 1 1 6028940F
-P 12800 8750
-F 0 "#PWR0144" H 12800 8500 50  0001 C CNN
-F 1 "GND" H 12805 8577 50  0000 C CNN
-F 2 "" H 12800 8750 50  0001 C CNN
-F 3 "" H 12800 8750 50  0001 C CNN
-	1    12800 8750
+P 12800 9050
+F 0 "#PWR0144" H 12800 8800 50  0001 C CNN
+F 1 "GND" H 12805 8877 50  0000 C CNN
+F 2 "" H 12800 9050 50  0001 C CNN
+F 3 "" H 12800 9050 50  0001 C CNN
+	1    12800 9050
 	1    0    0    -1
 $EndComp
@@
 L power:GND #PWR0110
 U 1 1 602F5C60
-P 8250 2450
-F 0 "#PWR0110" H 8250 2200 50  0001 C CNN
-F 1 "GND" H 8255 2277 50  0000 C CNN
-F 2 "" H 8250 2450 50  0001 C CNN
-F 3 "" H 8250 2450 50  0001 C CNN
-	1    8250 2450
+P 8250 2850
+F 0 "#PWR0110" H 8250 2600 50  0001 C CNN
+F 1 "GND" H 8255 2677 50  0000 C CNN
+F 2 "" H 8250 2850 50  0001 C CNN
+F 3 "" H 8250 2850 50  0001 C CNN
+	1    8250 2850
 	1    0    0    -1
 $EndComp
@@
 	1    0    0    -1
 $EndComp
+$Comp
+L Device:C C111
+U 1 1 624AD2F5
+P 8250 2600
+F 0 "C111" H 8365 2646 50  0000 L CNN
+F 1 "100nF" H 8365 2555 50  0000 L CNN
+F 2 "Capacitor_SMD:C_0402_1005Metric" H 8288 2450 50  0001 C CNN
+F 3 "~" H 8250 2600 50  0001 C CNN
+	1    8250 2600
+	1    0    0    -1
+$EndComp
+Wire Wire Line
+	8250 2750 8250 2850
+$Comp
+L Device:C C112
+U 1 1 624B7B96
+P 12800 8900
+F 0 "C112" H 12915 8946 50  0000 L CNN
+F 1 "100nF" H 12915 8855 50  0000 L CNN
+F 2 "Capacitor_SMD:C_0402_1005Metric" H 12838 8750 50  0001 C CNN
+F 3 "~" H 12800 8900 50  0001 C CNN
+	1    12800 8900
+	1    0    0    -1
+$EndComp
