File: KiCad/Proyecto_Final/Transceptor.sch (KiCad schematic (older format))
At the start: 33 parts, among them P1 SMA-KIT-1.5MF, T1 Input Balun, T2 output Balun, U1 hackrf_MAX2837

Commit message: avances en el esquemático
Parts:
- removed C10, C11: 3pF, symbol Device:C
- removed C?: 1000pF, symbol Device:C
- removed P1, P?: SMA-KIT-1.5MF, symbol gsg-symbols:SMA-KIT-1.5MF
- removed T2: output Balun, symbol hackrf:hackrf_BALUN
- removed TP?: TestPoint, symbol Connector:TestPoint
- added C?: 33pF, symbol Device:C
- added C?: 47pF, symbol Device:C
- added C? (x3): 10nF, symbol Device:C
- added C? (x2): 180pF, symbol Device:C
- added C?: 1uF, symbol Device:C
- added C?: 100pF, symbol Device:C
- added C? (x4): 100nF, symbol Device:C
- added R? (x2): 475, symbol Device:R
- added R? (x7): 0, symbol Device:R
- added U?: hackrf_SI5351C, symbol hackrf:hackrf_SI5351C
- added U?: hackrf_MAX5864, symbol hackrf:hackrf_MAX5864
Connections:
- net labels added: CSB, DIN, DOUT, ENABLE, RF_IN, RSSI, RXENABLE, RXHP, TXENABLE, VCCCP, VCCPLL, VCCRXBB1, VCCRXBB2, VCCRXMX, VCCVCO, VCCXTAL
- wire segments 74 -> 175
Other:
- note added: "Pines 42 43 44 45 --> Para TX (no usamos)"
- note added: "Recordar revisar etiquetas de tensiones, especialmente hasta el pin 18. \nDesde el pin 18 en adelante uso los nombres del kit de evaluación del MAX2837 (mucha documentación para evacuar dudas)"
- note removed: "Opción de referencia C"

Commit message: trabajo en el esquemático, MAX1193
Parts:
- removed U?: hackrf_MAX5864, symbol hackrf:hackrf_MAX5864
- added C? (x4): 2.2uF, symbol Device:C
- added C? (x4): 0.1uF, symbol Device:C
- added C? (x3): 0.33uF, symbol Device:C
- added U?: MAX1193ETI+, 21-0140L_T2855-3_MXM, symbol MAX1193:MAX1193ETI+
Connections:
- net labels added: GND1193, INA+, INA-, INB+, INB-, VDD
- wire segments 175 -> 211

Commit message: perifericos SI5351C
Parts:
- removed C?: 33pF, symbol Device:C
- added C? (x3): 47pF, symbol Device:C
- added C?: 1pF, symbol Device:C
- added R? (x3): 2k, symbol Device:R
- added R?: 10k, symbol Device:R
- added R? (x2): 0, symbol Device:R
- added X?: hackrf_GSG-XTAL4PIN, symbol hackrf:hackrf_GSG-XTAL4PIN
- C?: value 47pF -> 1pF
Connections:
- net labels added: 3v3, CLK_45Mhz, I2C_clock_in, I2C_data_in, Interrupt_Pin, MCU_CLK
- wire segments 211 -> 238
Other:
- note added: "Salidas D0 - D7 irian derecho al Micro si la velocidad\nde este es mayor"

Commit message: etiquetas y pines max2837
Parts:
- removed TP? (x6): TestPoint, symbol Connector:TestPoint
- added R?: 100, symbol Device:R
Connections:
- net labels added: VCC_LNA, VCC_PAD
- wire segments 238 -> 239
- no-connect marks 3 -> 9
Other:
- moved on the sheet: C?
Changed lines of the file:
@@
 	3650 2750 3400 2750
 Connection ~ 3400 2750
-$Comp
-L power:VAA #PWR0108
-U 1 1 5FDE3F56
-P 3950 3750
-F 0 "#PWR0108" H 3950 3600 50  0001 C CNN
-F 1 "VAA" V 3965 3877 50  0000 L CNN
-F 2 "" H 3950 3750 50  0001 C CNN
-F 3 "" H 3950 3750 50  0001 C CNN
-	1    3950 3750
-	0    -1   -1   0
-$EndComp
 NoConn ~ 6950 3450
 NoConn ~ 6950 3350
@@
 Wire Wire Line
 	4250 2900 4250 3150
-Wire Wire Line
-	4250 2750 4250 2900
-Connection ~ 4250 2900
-$Comp
-L Connector:TestPoint TP?
-U 1 1 6025CDB8
-P 3750 2200
-F 0 "TP?" H 3808 2318 50  0000 L CNN
-F 1 "TestPoint" H 3808 2227 50  0000 L CNN
-F 2 "" H 3950 2200 50  0001 C CNN
-F 3 "~" H 3950 2200 50  0001 C CNN
-	1    3750 2200
-	1    0    0    -1
-$EndComp
-Wire Wire Line
-	3750 3350 4350 3350
-Wire Wire Line
-	3750 2200 3750 3350
-Wire Wire Line
-	4350 3650 4000 3650
-$Comp
-L power:VCC #PWR0105
-U 1 1 6026E886
-P 4250 2750
-F 0 "#PWR0105" H 4250 2600 50  0001 C CNN
-F 1 "VCC" H 4265 2923 50  0000 C CNN
-F 2 "" H 4250 2750 50  0001 C CNN
-F 3 "" H 4250 2750 50  0001 C CNN
-	1    4250 2750
-	1    0    0    -1
-$EndComp
-Wire Wire Line
-	4350 3750 4050 3750
 $Comp
 L Device:C C?
 U 1 1 602785CE
-P 3250 3950
-F 0 "C?" V 2998 3950 50  0000 C CNN
-F 1 "22pF" V 3089 3950 50  0000 C CNN
-F 2 "" H 3288 3800 50  0001 C CNN
-F 3 "~" H 3250 3950 50  0001 C CNN
-	1    3250 3950
-	0    -1   -1   0
-$EndComp
-Wire Wire Line
-	4050 3750 4050 3950
-Wire Wire Line
-	4050 3950 3400 3950
-Connection ~ 4050 3750
-Wire Wire Line
-	4050 3750 3950 3750
+P 4000 3950
+F 0 "C?" V 3748 3950 50  0000 C CNN
+F 1 "22pF" V 3839 3950 50  0000 C CNN
+F 2 "" H 4038 3800 50  0001 C CNN
+F 3 "~" H 4000 3950 50  0001 C CNN
+	1    4000 3950
+	1    0    0    -1
+$EndComp
 $Comp
 L power:GND #PWR0107
 U 1 1 602890BB
-P 3100 3950
-F 0 "#PWR0107" H 3100 3700 50  0001 C CNN
-F 1 "GND" H 3105 3777 50  0000 C CNN
-F 2 "" H 3100 3950 50  0001 C CNN
-F 3 "" H 3100 3950 50  0001 C CNN
-	1    3100 3950
-	1    0    0    -1
-$EndComp
-$Comp
-L Connector:TestPoint TP?
-U 1 1 6028A1BE
-P 4300 3850
-F 0 "TP?" V 4350 4000 50  0000 C CNN
-F 1 "TestPoint" V 4350 3750 50  0000 C CNN
-F 2 "" H 4500 3850 50  0001 C CNN
-F 3 "~" H 4500 3850 50  0001 C CNN
-	1    4300 3850
-	0    -1   -1   0
-$EndComp
-$Comp
-L Connector:TestPoint TP?
-U 1 1 6028A932
-P 4300 3950
-F 0 "TP?" V 4350 4100 50  0000 C CNN
-F 1 "TestPoint" V 4350 3850 50  0000 C CNN
-F 2 "" H 4500 3950 50  0001 C CNN
-F 3 "~" H 4500 3950 50  0001 C CNN
-	1    4300 3950
-	0    -1   -1   0
-$EndComp
-Wire Wire Line
-	4350 3950 4300 3950
-Wire Wire Line
-	4350 3850 4300 3850
-$Comp
-L Connector:TestPoint TP?
-U 1 1 6028D003
-P 4350 4250
-F 0 "TP?" V 4400 4400 50  0000 C CNN
-F 1 "TestPoint" V 4400 4150 50  0000 C CNN
-F 2 "" H 4550 4250 50  0001 C CNN
-F 3 "~" H 4550 4250 50  0001 C CNN
-	1    4350 4250
-	0    -1   -1   0
-$EndComp
-$Comp
-L Connector:TestPoint TP?
-U 1 1 602902B6
-P 4750 5050
-F 0 "TP?" V 4800 5200 50  0000 C CNN
-F 1 "TestPoint" V 4800 4950 50  0000 C CNN
-F 2 "" H 4950 5050 50  0001 C CNN
-F 3 "~" H 4950 5050 50  0001 C CNN
-	1    4750 5050
-	0    -1   -1   0
+P 4000 4100
+F 0 "#PWR0107" H 4000 3850 50  0001 C CNN
+F 1 "GND" H 4005 3927 50  0000 C CNN
+F 2 "" H 4000 4100 50  0001 C CNN
+F 3 "" H 4000 4100 50  0001 C CNN
+	1    4000 4100
+	1    0    0    -1
 $EndComp
 $Comp
@@
 $EndComp
 Wire Wire Line
-	4750 5050 5200 5050
-Wire Wire Line
-	5200 5050 5200 5000
-Wire Wire Line
 	4400 5150 5300 5150
 Wire Wire Line
 	5300 5150 5300 5000
-$Comp
-L Connector:TestPoint TP?
-U 1 1 6029859C
-P 3850 5150
-F 0 "TP?" V 3900 5300 50  0000 C CNN
-F 1 "TestPoint" V 3900 5050 50  0000 C CNN
-F 2 "" H 4050 5150 50  0001 C CNN
-F 3 "~" H 4050 5150 50  0001 C CNN
-	1    3850 5150
-	0    -1   -1   0
-$EndComp
-Wire Wire Line
-	3850 5150 4000 5150
 $Comp
 L Device:R R?
@@
 Wire Wire Line
 	4000 4950 4000 5150
-Connection ~ 4000 5150
 Wire Wire Line
 	4000 5150 4100 5150
@@
 Wire Wire Line
 	4850 6100 5000 6100
+$Comp
+L power:GND #PWR?
+U 1 1 6030CF99
+P 4350 2800
+F 0 "#PWR?" H 4350 2550 50  0001 C CNN
+F 1 "GND" V 4355 2672 50  0000 R CNN
+F 2 "" H 4350 2800 50  0001 C CNN
+F 3 "" H 4350 2800 50  0001 C CNN
+	1    4350 2800
+	1    0    0    -1
+$EndComp
+NoConn ~ 4350 3350
+NoConn ~ 4350 3650
+NoConn ~ 4350 3850
+NoConn ~ 4350 3950
+Text GLabel 3950 3750 0    50   Input ~ 0
+VCC_PAD
+NoConn ~ 4350 4250
+Text GLabel 4250 2700 1    50   Input ~ 0
+VCC_LNA
+Wire Wire Line
+	4250 2700 4250 2900
+Connection ~ 4250 2900
+Wire Wire Line
+	3950 3750 4000 3750
+Wire Wire Line
+	4000 3800 4000 3750
+Connection ~ 4000 3750
+Wire Wire Line
+	4000 3750 4350 3750
+$Comp
+L Device:R R?
+U 1 1 60373025
+P 4200 4100
+F 0 "R?" H 4350 4100 50  0000 R CNN
+F 1 "100" V 4200 4150 50  0000 R CNN
+F 2 "" V 4130 4100 50  0001 C CNN
+F 3 "~" H 4200 4100 50  0001 C CNN
+	1    4200 4100
+	-1   0    0    1
+$EndComp
+Wire Wire Line
+	4300 3950 4300 4050
+Wire Wire Line
+	4300 4050 4350 4050
+Wire Wire Line
+	4200 3950 4300 3950
+Wire Wire Line
+	4350 4150 4300 4150
+Wire Wire Line
+	4300 4150 4300 4250
+Wire Wire Line
+	4300 4250 4200 4250
+$Comp
+L power:GND #PWR?
+U 1 1 603932CA
+P 4900 4800
+F 0 "#PWR?" H 4900 4550 50  0001 C CNN
+F 1 "GND" H 4905 4627 50  0000 C CNN
+F 2 "" H 4900 4800 50  0001 C CNN
+F 3 "" H 4900 4800 50  0001 C CNN
+	1    4900 4800
+	1    0    0    -1
+$EndComp
+Wire Wire Line
+	5100 5000 5000 5000
+Wire Wire Line
+	5000 5000 5000 4750
+Wire Wire Line
+	5000 4750 4900 4750
+Wire Wire Line
+	4900 4750 4900 4800
+NoConn ~ 5200 5000
 $EndSCHEMATC

Commit message: tranceptor esquematico completo
Parts:
- removed C1, C14, C2, C3: 22p, symbol Device:C
- removed C12, C13, C4, C5: 10n, symbol Device:C
- removed C6: 100p, symbol Device:C
- removed C9: 100n, symbol Device:C
- removed C?: 100pF, symbol Device:C
- removed P?: SMA-KIT-1.5MF, symbol gsg-symbols:SMA-KIT-1.5MF
- removed R? (x6): 0, symbol Device:R
- removed T1: Input Balun, symbol hackrf:hackrf_BALUN
- added C?: 50pF, symbol Device:C
- added C?: 0.1uF, symbol Device:C
- added T?: 2450BL05A0100, Tesis2020-21:0202_Balun, symbol Tesis2020-21:2450BL05A0100
- C? (x2): value 100nF -> 10nF
- C?: value 100nF -> 22pF
- U1: footprint Maxim:MAX2837ETM&plus_ -> footprints:MAX2837ETM&plus_
- U?: footprint 21-0140L_T2855-3_MXM -> max1193pretty:MAX1193ETI&plus_T
Connections:
- net labels added: A_B, D0, D1, D2, D3, D4, D5, D6, D7, PD0, PD1
- net labels removed: CLK_OUT, RXHP, VAA, VCCCP, VCCPLL, VCCRXBB1, VCCRXBB2, VCCRXMX, VCCVCO, VCCXTAL, VCC_LNA, VCC_PAD
- wire segments 239 -> 198
- no-connect marks 9 -> 10
Other:
- note added: "DUDAS:\n\n1. Pines B0-B7 a masa? se usan? \nMaximum gain, B7:B1 = 0000000 \nMinimum gain, B7:B1 = 1111111\n\n2. Pin 7 VCCTXPAD ver\n\n3. Pines 10 y 11 ver\n\n4. Pin 13 está bien a GND?\n\n5. Pin 16 ver\n\n6. Pines 42 43 44 45 Cuál es la opción de menos ruido? GND? soldado al pad?"
- note added: "Pines 13 al 23 van al micro"
- note removed: "Recordar revisar etiquetas de tensiones, especialmente hasta el pin 18. \nDesde el pin 18 en adelante uso los nombres del kit de evaluación del MAX2837 (mucha documentación para evacuar dudas)"
- note removed: "Salidas D0 - D7 irian derecho al Micro si la velocidad\nde este es mayor"
- moved on the sheet: C?

Commit message: Actualización hoja MCU y latex.
Parts:
- removed C? (x2): 1pF, symbol Device:C
- removed C? (x3): 47pF, symbol Device:C
- removed C?: 50pF, symbol Device:C
- removed R? (x3): 2k, symbol Device:R
- removed R?: 10k, symbol Device:R
- removed U?: hackrf_SI5351C, symbol hackrf:hackrf_SI5351C
- removed X?: hackrf_GSG-XTAL4PIN, symbol hackrf:hackrf_GSG-XTAL4PIN
- U?: symbol MAX1193:MAX1193ETI+ -> Transceptor-rescue:MAX1193ETI+-MAX1193
Connections:
- net labels removed: 3v3, I2C_clock_in, I2C_data_in, Interrupt_Pin, MCU_CLK, VCC
- wire segments 198 -> 163

Commit message: Cambio nombre de datasheets para búsqueda rápida, actualizada hoja MCU, modificadas hojas de frontend y transceptor.
Parts:
- added R?: 10k, symbol Device:R
Connections:
- net labels added: RF_IF
- net labels removed: RF_IN
- wire segments 163 -> 164
Changed lines of the file:
@@
 	5100 1950 5100 2400
 Text GLabel 1650 2350 0    50   Input ~ 0
-RF_IN
+RF_IF
 $Comp
 L Transceptor-rescue:MAX1193ETI+-MAX1193 U?
@@
 	-1   0    0    1
 $EndComp
+Text GLabel 3550 1150 0    50   Input ~ 0
+TXENABLE
+$Comp
+L Device:R R?
+U 1 1 6072CDC3
+P 3650 1300
+F 0 "R?" H 3720 1346 50  0000 L CNN
+F 1 "10k" H 3720 1255 50  0000 L CNN
+F 2 "" V 3580 1300 50  0001 C CNN
+F 3 "~" H 3650 1300 50  0001 C CNN
+	1    3650 1300
+	1    0    0    -1
+$EndComp
+Wire Wire Line
+	3550 1150 3650 1150
+$Comp
+L power:GND #PWR?
+U 1 1 607344AB
+P 3650 1450
+F 0 "#PWR?" H 3650 1200 50  0001 C CNN
+F 1 "GND" H 3655 1277 50  0000 C CNN
+F 2 "" H 3650 1450 50  0001 C CNN
+F 3 "" H 3650 1450 50  0001 C CNN
+	1    3650 1450
+	1    0    0    -1
+$EndComp
 $EndSCHEMATC

Commit message: Update hoja MCU y transceptor.
Connections:
- net labels added: SPI1_CS1, SPI1_MISO, SPI1_MOSI, SPI1_SCK, Trx_Enable, Trx_Rx_Enable
- net labels removed: CSB, DIN, DOUT, ENABLE, RXENABLE, SCLK
- wire segments 164 -> 160
Changed lines of the file:
@@
 	5300 5150 5300 5000
 Text GLabel 3900 4950 0    50   Input ~ 0
-SCLK
+SPI1_SCK
 Wire Wire Line
 	3900 4950 4000 4950
@@
 Connection ~ 7400 5250
 Text GLabel 6950 4550 3    50   Input ~ 0
-ENABLE
+Trx_Enable
 Wire Wire Line
 	6950 4550 6950 4250
@@
 Text GLabel 8300 3950 2    50   Input ~ 0
 VDD
-Text GLabel 8700 3850 2    50   Input ~ 0
-DOUT
-Text GLabel 7550 3750 2    50   Input ~ 0
-CSB
-Text GLabel 7750 3650 2    50   Input ~ 0
-DIN
-Text GLabel 7100 3550 2    50   Input ~ 0
+Text GLabel 6950 3850 2    50   Input ~ 0
+SPI1_MISO
+Text GLabel 6950 3750 2    50   Input ~ 0
+SPI1_CS1
+Text GLabel 6950 3650 2    50   Input ~ 0
+SPI1_MOSI
+Text GLabel 6950 3550 2    50   Input ~ 0
 RSSI
 $Comp
@@
 TXENABLE
 Text GLabel 4850 1950 0    50   Input ~ 0
-RXENABLE
+Trx_Rx_Enable
 Wire Wire Line
 	5100 1750 5200 1750
@@
 Wire Wire Line
 	7750 3950 8300 3950
-Wire Wire Line
-	6950 3850 8700 3850
-Wire Wire Line
-	6950 3750 7550 3750
-Wire Wire Line
-	7750 3650 6950 3650
-Wire Wire Line
-	6950 3550 7100 3550
 NoConn ~ 5900 2400
 Wire Wire Line
