File: KiCad/Proyecto_Final/Transceptor.sch (KiCad schematic (older format))
At the start: 39 parts, among them U1 hackrf_MAX2837

Commit message: Update esquemático, reubicación de archivos Gantt.
Parts:
- removed C?: 0.1uF, symbol Device:C
- removed R? (x5): 0, symbol Device:R
- added C?: 22pF, symbol Device:C
- added C? (x2): 10pF, symbol Device:C
- added R? (x4): 10k, symbol Device:R
- added Y?: 40MHz, symbol Device:Crystal_GND24
Connections:
- net GND1193 is gone; now on net GND: U?.3 (GND)
- net GND: now also C?.2, C?.2, C?.2, R?.2, R?.2, R?.2, R?.2, Y?.2, Y?.4; no longer U1.13 (VCCTXMX), U1.42 (TXBBI-), U1.43 (TXBBI+), U1.44 (TXBBQ+), U1.45 (TXBBQ-)
- net INA+: now also U1.38 (RXBBI+)
- net INA-: now also U1.37 (RXBBI-)
- net INB+: now also U1.36 (RXBBQ+)
- net INB-: now also U1.35 (RXBBQ-)
- net SPI1_SCK: now also U1.15 (SCLK)
- net B1: now reaches U1.12 (B1)
- net XTAL2: now reaches U1.17 (XTAL2)
- net XTAL2: now also C?.1, Y?.1
- net XTAL1: now reaches U1.18 (XTAL1)
- net XTAL1: now also C?.1, Y?.3
- net B5: now reaches U1.3 (B5)
- net B7: now reaches U1.33 (B7)
- net B6: now reaches U1.34 (B6)
- net RXHP: now reaches U1.40 (RXHP)
- net B4: now reaches U1.6 (B4)
- net B3: now reaches U1.8 (B3)
- net B2: now reaches U1.9 (B2)
- net CLK_45Mhz renamed CLK_ADC
- net VDD renamed +3V3
- net +3V3: now also U1.13 (VCCTXMX), C?.1
- new net TXBBI+: R?.1, U1.43 (TXBBI+)
- new net TXBBI-: R?.1, U1.42 (TXBBI-)
- new net TXBBQ+: R?.1, U1.44 (TXBBQ+)
- new net TXBBQ-: R?.1, U1.45 (TXBBQ-)
- no-connect marks 10 -> 3
Other:
- note removed: "DUDAS:\n\n1. Pines B0-B7 a masa? se usan? \nMaximum gain, B7:B1 = 0000000 \nMinimum gain, B7:B1 = 1111111\n\n2. Pin 7 VCCTXPAD ver\n\n3. Pines 10 y 11 ver\n\n4. Pin 13 está bien a GND?\n\n5. Pin 16 ver\n\n6. Pines 42 43 44 45 Cuál es la opción de menos ruido? GND? soldado al pad?"
- note removed: "Pines 13 al 23 van al micro"
- note removed: "Pines 42 43 44 45 --> Para TX (no usamos)"
- moved on the sheet: C?, R?

Commit message: Terminado esquematico.
Parts:
- removed C? (x2): 10pF, symbol Device:C
- removed Y?: 40MHz, symbol Device:Crystal_GND24
- added C?: 1nF, symbol Device:C
- added J?: ADC_CLK_SEL, symbol Connector_Generic:Conn_02x02_Counter_Clockwise
Connections:
- net CLK_ADC: now also J?.3 (Pin_3), J?.4 (Pin_4)
- net XTAL2: now also C?.1
- net XTAL1: no longer names the net of U1.18 (XTAL1)
- new net ADC_22MHz: J?.1 (Pin_1)
- new net ADC_45MHz: J?.2 (Pin_2)
- new net Trx_CLK: C?.2
- no-connect marks 3 -> 4
Changed lines of the file:
@@
 Wire Wire Line
 	10400 5000 10500 5000
+NoConn ~ 5600 5000
 $Comp
-L Device:Crystal_GND24 Y?
-U 1 1 60752419
-P 5750 6950
-F 0 "Y?" H 5700 7350 50  0000 L CNN
-F 1 "40MHz" H 5600 7250 50  0000 L CNN
-F 2 "" H 5750 6950 50  0001 C CNN
-F 3 "~" H 5750 6950 50  0001 C CNN
-	1    5750 6950
+L Device:C C?
+U 1 1 60782802
+P 4200 6000
+F 0 "C?" V 3948 6000 50  0000 C CNN
+F 1 "1nF" V 4039 6000 50  0000 C CNN
+F 2 "" H 4238 5850 50  0001 C CNN
+F 3 "~" H 4200 6000 50  0001 C CNN
+	1    4200 6000
+	0    1    1    0
+$EndComp
+Text GLabel 5500 5000 3    50   Input ~ 0
+XTAL2
+Text GLabel 4500 6000 2    50   Input ~ 0
+XTAL2
+Text GLabel 3900 6000 0    50   Input ~ 0
+Trx_CLK
+Wire Wire Line
+	3900 6000 4050 6000
+Wire Wire Line
+	4350 6000 4500 6000
+Text GLabel 13850 4750 2    50   Input ~ 0
+CLK_ADC
+$Comp
+L Connector_Generic:Conn_02x02_Counter_Clockwise J?
+U 1 1 6079C663
+P 13400 4750
+F 0 "J?" H 13450 4967 50  0000 C CNN
+F 1 "ADC_CLK_SEL" H 13450 4876 50  0000 C CNN
+F 2 "" H 13400 4750 50  0001 C CNN
+F 3 "~" H 13400 4750 50  0001 C CNN
+	1    13400 4750
 	1    0    0    -1
 $EndComp
 Wire Wire Line
-	5750 6750 5750 6700
+	13700 4750 13850 4750
 Wire Wire Line
-	5750 6700 5500 6700
+	13700 4850 13700 4750
+Connection ~ 13700 4750
+Text GLabel 13050 4750 0    50   Input ~ 0
+ADC_22MHz
+Text GLabel 13050 4850 0    50   Input ~ 0
+ADC_45MHz
 Wire Wire Line
-	5500 6700 5500 7200
+	13050 4750 13200 4750
 Wire Wire Line
-	5500 7200 5750 7200
-Wire Wire Line
-	5750 7200 5750 7150
-$Comp
-L power:GND #PWR?
-U 1 1 607596F3
-P 5750 7200
-F 0 "#PWR?" H 5750 6950 50  0001 C CNN
-F 1 "GND" H 5755 7027 50  0000 C CNN
-F 2 "" H 5750 7200 50  0001 C CNN
-F 3 "" H 5750 7200 50  0001 C CNN
-	1    5750 7200
-	1    0    0    -1
-$EndComp
-Connection ~ 5750 7200
-$Comp
-L Device:C C?
-U 1 1 6075A834
-P 5200 7100
-F 0 "C?" H 5315 7146 50  0000 L CNN
-F 1 "10pF" H 5315 7055 50  0000 L CNN
-F 2 "" H 5238 6950 50  0001 C CNN
-F 3 "~" H 5200 7100 50  0001 C CNN
-	1    5200 7100
-	1    0    0    -1
-$EndComp
-$Comp
-L Device:C C?
-U 1 1 6075B1C0
-P 6100 7100
-F 0 "C?" H 6215 7146 50  0000 L CNN
-F 1 "10pF" H 6215 7055 50  0000 L CNN
-F 2 "" H 6138 6950 50  0001 C CNN
-F 3 "~" H 6100 7100 50  0001 C CNN
-	1    6100 7100
-	1    0    0    -1
-$EndComp
-$Comp
-L power:GND #PWR?
-U 1 1 6075BE55
-P 5200 7250
-F 0 "#PWR?" H 5200 7000 50  0001 C CNN
-F 1 "GND" H 5205 7077 50  0000 C CNN
-F 2 "" H 5200 7250 50  0001 C CNN
-F 3 "" H 5200 7250 50  0001 C CNN
-	1    5200 7250
-	1    0    0    -1
-$EndComp
-$Comp
-L power:GND #PWR?
-U 1 1 6075C135
-P 6100 7250
-F 0 "#PWR?" H 6100 7000 50  0001 C CNN
-F 1 "GND" H 6105 7077 50  0000 C CNN
-F 2 "" H 6100 7250 50  0001 C CNN
-F 3 "" H 6100 7250 50  0001 C CNN
-	1    6100 7250
-	1    0    0    -1
-$EndComp
-Wire Wire Line
-	5200 6950 5600 6950
-Wire Wire Line
-	5900 6950 6100 6950
-Text GLabel 5600 5000 3    50   Input ~ 0
-XTAL1
-Text GLabel 5500 5000 3    50   Input ~ 0
-XTAL2
-Text GLabel 5100 6950 0    50   Input ~ 0
-XTAL2
-Wire Wire Line
-	5100 6950 5200 6950
-Connection ~ 5200 6950
-Text GLabel 6200 6950 2    50   Input ~ 0
-XTAL1
-Wire Wire Line
-	6200 6950 6100 6950
-Connection ~ 6100 6950
+	13050 4850 13200 4850
 $EndSCHEMATC

Commit message: Esquematico terminado con test points.
Parts:
- added R? (x4): 0, symbol Device:R
- added TP? (x11): TestPoint, symbol Connector:TestPoint
Connections:
- net A_B: now also TP?.1
- net D0: now also TP?.1
- net D1: now also TP?.1
- net D2: now also TP?.1
- net D3: now also TP?.1
- net D4: now also TP?.1
- net D5: now also TP?.1
- net D6: now also TP?.1
- net D7: now also TP?.1
- net INA+: now also R?.2; no longer U?.2 (INA+)
- net INA-: now also R?.2; no longer U?.1 (INA-)
- net INB+: now also R?.2; no longer U?.6 (INB+)
- net INB-: now also R?.2; no longer U?.7 (INB-)
- net PD0: now also TP?.1
- net PD1: now also TP?.1
- new net _INA+: R?.1, U?.2 (INA+)
- new net _INA-: R?.1, U?.1 (INA-)
- new net _INB+: R?.1, U?.6 (INB+)
- new net _INB-: R?.1, U?.7 (INB-)
Other:
- note added: "Separadores para medición"
Changed lines of the file:
@@
 Text GLabel 6950 3250 2    50   Input ~ 0
 INB-
-Text GLabel 12300 1950 0    50   Input ~ 0
-INA-
-Text GLabel 12300 2050 0    50   Input ~ 0
-INA+
-Text GLabel 12300 2550 0    50   Input ~ 0
-INB-
-Text GLabel 12300 2450 0    50   Input ~ 0
-INB+
 Wire Wire Line
 	10950 1950 10950 2050
@@
 Wire Wire Line
 	13050 4850 13200 4850
+$Comp
+L Device:R R?
+U 1 1 60791BA0
+P 8650 1700
+F 0 "R?" V 8443 1700 50  0000 C CNN
+F 1 "0" V 8534 1700 50  0000 C CNN
+F 2 "" V 8580 1700 50  0001 C CNN
+F 3 "~" H 8650 1700 50  0001 C CNN
+	1    8650 1700
+	0    1    1    0
+$EndComp
+$Comp
+L Device:R R?
+U 1 1 60798900
+P 8650 2050
+F 0 "R?" V 8443 2050 50  0000 C CNN
+F 1 "0" V 8534 2050 50  0000 C CNN
+F 2 "" V 8580 2050 50  0001 C CNN
+F 3 "~" H 8650 2050 50  0001 C CNN
+	1    8650 2050
+	0    1    1    0
+$EndComp
+$Comp
+L Device:R R?
+U 1 1 60798B8E
+P 8650 2400
+F 0 "R?" V 8443 2400 50  0000 C CNN
+F 1 "0" V 8534 2400 50  0000 C CNN
+F 2 "" V 8580 2400 50  0001 C CNN
+F 3 "~" H 8650 2400 50  0001 C CNN
+	1    8650 2400
+	0    1    1    0
+$EndComp
+$Comp
+L Device:R R?
+U 1 1 60798F18
+P 8650 2750
+F 0 "R?" V 8443 2750 50  0000 C CNN
+F 1 "0" V 8534 2750 50  0000 C CNN
+F 2 "" V 8580 2750 50  0001 C CNN
+F 3 "~" H 8650 2750 50  0001 C CNN
+	1    8650 2750
+	0    1    1    0
+$EndComp
+Text GLabel 8500 1700 0    50   Input ~ 0
+INA+
+Text GLabel 8500 2050 0    50   Input ~ 0
+INA-
+Text GLabel 8500 2400 0    50   Input ~ 0
+INB+
+Text GLabel 8500 2750 0    50   Input ~ 0
+INB-
+Text GLabel 8800 1700 2    50   Input ~ 0
+_INA+
+Text GLabel 8800 2050 2    50   Input ~ 0
+_INA-
+Text GLabel 8800 2400 2    50   Input ~ 0
+_INB+
+Text GLabel 8800 2750 2    50   Input ~ 0
+_INB-
+Text GLabel 12300 2050 0    50   Input ~ 0
+_INA+
+Text GLabel 12300 1950 0    50   Input ~ 0
+_INA-
+Text GLabel 12300 2450 0    50   Input ~ 0
+_INB+
+Text GLabel 12300 2550 0    50   Input ~ 0
+_INB-
+Wire Notes Line
+	8200 1400 8200 2850
+Wire Notes Line
+	8200 2850 9150 2850
+Wire Notes Line
+	9150 2850 9150 1400
+Wire Notes Line
+	9150 1400 8200 1400
+Text Notes 8200 1350 0    50   ~ 0
+Separadores para medición
+Text GLabel 14550 4250 3    50   Input ~ 0
+D5
+Text GLabel 14700 4250 3    50   Input ~ 0
+D4
+Text GLabel 15750 4250 3    50   Input ~ 0
+A_B
+Text GLabel 14850 4250 3    50   Input ~ 0
+D3
+Text GLabel 15000 4250 3    50   Input ~ 0
+D2
+Text GLabel 15150 4250 3    50   Input ~ 0
+D1
+Text GLabel 15300 4250 3    50   Input ~ 0
+D0
+Text GLabel 15450 4250 3    50   Input ~ 0
+PD1
+Text GLabel 15600 4250 3    50   Input ~ 0
+PD0
+$Comp
+L Connector:TestPoint TP?
+U 1 1 607AE5A5
+P 14550 4250
+F 0 "TP?" H 14500 4450 50  0000 L CNN
+F 1 "TestPoint" H 14350 4600 50  0001 L CNN
+F 2 "" H 14750 4250 50  0001 C CNN
+F 3 "~" H 14750 4250 50  0001 C CNN
+	1    14550 4250
+	1    0    0    -1
+$EndComp
+$Comp
+L Connector:TestPoint TP?
+U 1 1 607C1A8B
+P 14700 4250
+F 0 "TP?" H 14650 4450 50  0000 L CNN
+F 1 "TestPoint" H 14500 4600 50  0001 L CNN
+F 2 "" H 14900 4250 50  0001 C CNN
+F 3 "~" H 14900 4250 50  0001 C CNN
+	1    14700 4250
+	1    0    0    -1
+$EndComp
+$Comp
+L Connector:TestPoint TP?
+U 1 1 607DFB6E
+P 15750 4250
+F 0 "TP?" H 15700 4450 50  0000 L CNN
+F 1 "TestPoint" H 15550 4600 50  0001 L CNN
+F 2 "" H 15950 4250 50  0001 C CNN
+F 3 "~" H 15950 4250 50  0001 C CNN
+	1    15750 4250
+	1    0    0    -1
+$EndComp
+$Comp
+L Connector:TestPoint TP?
+U 1 1 607DFE0C
+P 14850 4250
+F 0 "TP?" H 14800 4450 50  0000 L CNN
+F 1 "TestPoint" H 14650 4600 50  0001 L CNN
+F 2 "" H 15050 4250 50  0001 C CNN
+F 3 "~" H 15050 4250 50  0001 C CNN
+	1    14850 4250
+	1    0    0    -1
+$EndComp
+$Comp
+L Connector:TestPoint TP?
+U 1 1 607DFFDB
+P 15000 4250
+F 0 "TP?" H 14950 4450 50  0000 L CNN
+F 1 "TestPoint" H 14800 4600 50  0001 L CNN
+F 2 "" H 15200 4250 50  0001 C CNN
+F 3 "~" H 15200 4250 50  0001 C CNN
+	1    15000 4250
+	1    0    0    -1
+$EndComp
+$Comp
+L Connector:TestPoint TP?
+U 1 1 607E00F5
+P 15150 4250
+F 0 "TP?" H 15100 4450 50  0000 L CNN
+F 1 "TestPoint" H 14950 4600 50  0001 L CNN
+F 2 "" H 15350 4250 50  0001 C CNN
+F 3 "~" H 15350 4250 50  0001 C CNN
+	1    15150 4250
+	1    0    0    -1
+$EndComp
+$Comp
+L Connector:TestPoint TP?
+U 1 1 607E0392
+P 15300 4250
+F 0 "TP?" H 15250 4450 50  0000 L CNN
+F 1 "TestPoint" H 15100 4600 50  0001 L CNN
+F 2 "" H 15500 4250 50  0001 C CNN
+F 3 "~" H 15500 4250 50  0001 C CNN
+	1    15300 4250
+	1    0    0    -1
+$EndComp
+$Comp
+L Connector:TestPoint TP?
+U 1 1 607E0698
+P 15450 4250
+F 0 "TP?" H 15400 4450 50  0000 L CNN
+F 1 "TestPoint" H 15250 4600 50  0001 L CNN
+F 2 "" H 15650 4250 50  0001 C CNN
+F 3 "~" H 15650 4250 50  0001 C CNN
+	1    15450 4250
+	1    0    0    -1
+$EndComp
+$Comp
+L Connector:TestPoint TP?
+U 1 1 607E08DA
+P 15600 4250
+F 0 "TP?" H 15550 4450 50  0000 L CNN
+F 1 "TestPoint" H 15400 4600 50  0001 L CNN
+F 2 "" H 15800 4250 50  0001 C CNN
+F 3 "~" H 15800 4250 50  0001 C CNN
+	1    15600 4250
+	1    0    0    -1
+$EndComp
+Text GLabel 14250 4250 3    50   Input ~ 0
+D7
+Text GLabel 14400 4250 3    50   Input ~ 0
+D6
+$Comp
+L Connector:TestPoint TP?
+U 1 1 607E6856
+P 14400 4250
+F 0 "TP?" H 14350 4450 50  0000 L CNN
+F 1 "TestPoint" H 14200 4600 50  0001 L CNN
+F 2 "" H 14600 4250 50  0001 C CNN
+F 3 "~" H 14600 4250 50  0001 C CNN
+	1    14400 4250
+	1    0    0    -1
+$EndComp
+$Comp
+L Connector:TestPoint TP?
+U 1 1 607E6ACC
+P 14250 4250
+F 0 "TP?" H 14200 4450 50  0000 L CNN
+F 1 "TestPoint" H 14050 4600 50  0001 L CNN
+F 2 "" H 14450 4250 50  0001 C CNN
+F 3 "~" H 14450 4250 50  0001 C CNN
+	1    14250 4250
+	1    0    0    -1
+$EndComp
 $EndSCHEMATC

Commit message: Primer hito presentado y visado.
Parts:
- U1: value hackrf_MAX2837 -> MAX2837
Changed lines of the file:
@@
 U 1 1 5FDA61AC
 P 5650 3700
-F 0 "U1" H 5650 3900 60  0000 L CNN
-F 1 "hackrf_MAX2837" H 5350 4000 60  0000 L CNN
+F 0 "U1" H 5600 3750 60  0000 L CNN
+F 1 "MAX2837" H 5450 3650 60  0000 L CNN
 F 2 "footprints:MAX2837ETM&plus_" H 5650 3700 60  0001 C CNN
 F 3 "" H 5650 3700 60  0000 C CNN

Commit message: Empezando con el pcb, loquita.
Parts:
- C49, C50, C51, C53, C55, C62, C65, C66, C67, C69, C70, C71, C72, C73, C74, C75: renamed from C?; footprint (none) -> Capacitor_SMD:C_0402_1005Metric
- C52, C54, C61, C64, C68: renamed from C?; footprint (none) -> Capacitor_SMD:C_0805_2012Metric
- C56: renamed from C7; footprint (none) -> Capacitor_SMD:C_0402_1005Metric
- C57, C59, C63: renamed from C?; footprint (none) -> Capacitor_SMD:C_0603_1608Metric
- C58: renamed from C8; footprint (none) -> Capacitor_SMD:C_0402_1005Metric
- C60: renamed from C15; footprint (none) -> Capacitor_SMD:C_0402_1005Metric
- J2: renamed from J?; footprint (none) -> Connector_PinHeader_2.54mm:PinHeader_2x02_P2.54mm_Vertical_SMD
- L4: renamed from L1; footprint (none) -> Inductor_SMD:L_0402_1005Metric
- R10, R11, R16, R17, R18, R7, R8, R9: renamed from R?; footprint (none) -> Resistor_SMD:R_0402_1005Metric
- R12, R13, R14, R15: renamed from R?; footprint (none) -> Resistor_SMD:R_0201_0603Metric
- gave numbers to parts that had none: 13
- renumbered U1 to U10

Commit message: Empezado PCB.
Parts:
- TP1, TP10, TP11, TP2, TP3, TP4, TP5, TP6, TP7, TP8, TP9: footprint (none) -> TestPoint:TestPoint_Pad_D1.0mm
Changed lines of the file:
@@
 F 0 "TP3" H 14500 4450 50  0000 L CNN
 F 1 "TestPoint" H 14350 4600 50  0001 L CNN
-F 2 "" H 14750 4250 50  0001 C CNN
+F 2 "TestPoint:TestPoint_Pad_D1.0mm" H 14750 4250 50  0001 C CNN
 F 3 "~" H 14750 4250 50  0001 C CNN
 	1    14550 4250
@@
 F 0 "TP4" H 14650 4450 50  0000 L CNN
 F 1 "TestPoint" H 14500 4600 50  0001 L CNN
-F 2 "" H 14900 4250 50  0001 C CNN
+F 2 "TestPoint:TestPoint_Pad_D1.0mm" H 14900 4250 50  0001 C CNN
 F 3 "~" H 14900 4250 50  0001 C CNN
 	1    14700 4250
@@
 F 0 "TP11" H 15700 4450 50  0000 L CNN
 F 1 "TestPoint" H 15550 4600 50  0001 L CNN
-F 2 "" H 15950 4250 50  0001 C CNN
+F 2 "TestPoint:TestPoint_Pad_D1.0mm" H 15950 4250 50  0001 C CNN
 F 3 "~" H 15950 4250 50  0001 C CNN
 	1    15750 4250
@@
 F 0 "TP5" H 14800 4450 50  0000 L CNN
 F 1 "TestPoint" H 14650 4600 50  0001 L CNN
-F 2 "" H 15050 4250 50  0001 C CNN
+F 2 "TestPoint:TestPoint_Pad_D1.0mm" H 15050 4250 50  0001 C CNN
 F 3 "~" H 15050 4250 50  0001 C CNN
 	1    14850 4250
@@
 F 0 "TP6" H 14950 4450 50  0000 L CNN
 F 1 "TestPoint" H 14800 4600 50  0001 L CNN
-F 2 "" H 15200 4250 50  0001 C CNN
+F 2 "TestPoint:TestPoint_Pad_D1.0mm" H 15200 4250 50  0001 C CNN
 F 3 "~" H 15200 4250 50  0001 C CNN
 	1    15000 4250
@@
 F 0 "TP7" H 15100 4450 50  0000 L CNN
 F 1 "TestPoint" H 14950 4600 50  0001 L CNN
-F 2 "" H 15350 4250 50  0001 C CNN
+F 2 "TestPoint:TestPoint_Pad_D1.0mm" H 15350 4250 50  0001 C CNN
 F 3 "~" H 15350 4250 50  0001 C CNN
 	1    15150 4250
@@
 F 0 "TP8" H 15250 4450 50  0000 L CNN
 F 1 "TestPoint" H 15100 4600 50  0001 L CNN
-F 2 "" H 15500 4250 50  0001 C CNN
+F 2 "TestPoint:TestPoint_Pad_D1.0mm" H 15500 4250 50  0001 C CNN
 F 3 "~" H 15500 4250 50  0001 C CNN
 	1    15300 4250
@@
 F 0 "TP9" H 15400 4450 50  0000 L CNN
 F 1 "TestPoint" H 15250 4600 50  0001 L CNN
-F 2 "" H 15650 4250 50  0001 C CNN
+F 2 "TestPoint:TestPoint_Pad_D1.0mm" H 15650 4250 50  0001 C CNN
 F 3 "~" H 15650 4250 50  0001 C CNN
 	1    15450 4250
@@
 F 0 "TP10" H 15550 4450 50  0000 L CNN
 F 1 "TestPoint" H 15400 4600 50  0001 L CNN
-F 2 "" H 15800 4250 50  0001 C CNN
+F 2 "TestPoint:TestPoint_Pad_D1.0mm" H 15800 4250 50  0001 C CNN
 F 3 "~" H 15800 4250 50  0001 C CNN
 	1    15600 4250
@@
 F 0 "TP2" H 14350 4450 50  0000 L CNN
 F 1 "TestPoint" H 14200 4600 50  0001 L CNN
-F 2 "" H 14600 4250 50  0001 C CNN
+F 2 "TestPoint:TestPoint_Pad_D1.0mm" H 14600 4250 50  0001 C CNN
 F 3 "~" H 14600 4250 50  0001 C CNN
 	1    14400 4250
@@
 F 0 "TP1" H 14200 4450 50  0000 L CNN
 F 1 "TestPoint" H 14050 4600 50  0001 L CNN
-F 2 "" H 14450 4250 50  0001 C CNN
+F 2 "TestPoint:TestPoint_Pad_D1.0mm" H 14450 4250 50  0001 C CNN
 F 3 "~" H 14450 4250 50  0001 C CNN
 	1    14250 4250

Commit message: Avance PCB.
Parts:
- removed R12, R13, R14, R15: 0, Resistor_SMD:R_0201_0603Metric, symbol Device:R
- renumbered R9 to R10, R10 to R11, R11 to R12, R16 to R13, R17 to R14, R18 to R15, R7 to R8, R8 to R9
Connections:
- net _INA+ is gone; now on net INA+: U9.2 (INA+)
- net _INA- is gone; now on net INA-: U9.1 (INA-)
- net _INB+ is gone; now on net INB+: U9.6 (INB+)
- net _INB- is gone; now on net INB-: U9.7 (INB-)
- net RXRF+: now reaches C56.1, L4.1, U10.4 (RXRF+)
- net RXRF-: now reaches C58.1, L4.2, U10.5 (RXRF-)
Other:
- note removed: "Separadores para medición"
